File: flight_tracker_prototype.kicad_sch (KiCad schematic)
At the start: 2 parts, among them J1 1.54" ST7789 LCD

Commit message: Added buzzer to schematic
Parts:
- added BZ1: Buzzer, symbol Device:Buzzer
Connections:
- net GND: now also BZ1.2 (-)
- net at A1.19 (GPIO14): now also BZ1.1 (+)
- no-connect marks 24 -> 23
Other:
- moved on the sheet: A1, J1
